File: hardware/TinySpectrometer-mk-1.0.sch (EAGLE design)
At the start: 11 parts, among them J1 DF12-32-DP-NOTREALLY, U1 GRIDEYE

Commit message: whole lotta commits
Parts:
- removed ADDR: (no value), a_parts:JUMPER-PAD-3-NOSMALLER
- added JP1, JP3: M04PTH-CENTERED, a_parts:M04PTH-CENTERED
- added JP2: M03PTH-CENTERED, a_parts:M03PTH-CENTERED
- added LED: LED1206, a_parts:LED1206
- added MEM: LED0603-TIGHT, a_parts:LED0603-TIGHT
- added R5: 10K, a_parts:RESISTORR0603-TIGHTER
- added U2: (no value), a_parts:SPI_FLASHSOIC
- C2: value 1u -> 100n
- C3: value 1u5 -> 1u
- J1: value DF12-32-DP-NOTREALLY -> (none); device a_parts:DF12-32-DP-NOTREALLY -> a_parts:JUMPER-PAD-3-NOSMALLER
- R3: value 10K -> DNP
- R4: value 20R -> 10K
- U1: value GRIDEYE -> AS7263; device a_parts:GRIDEYEFATTER -> a_parts:AS7263
Connections:
- removed net ADDR: ADDR.2, U1.ADDR
- new net !CS_EE: JP3.1, U1.!CSN_EE, U2.!CS
- new net !CS_SD: JP2.1, U1.!CSN_SD
- new net !RESET: JP2.3, R4.1, U1.!RESN
- new net I2C_ENB: J1.2, U1.I2C_EN
- new net MISO: JP3.2, U1.MISO, U2.MISO
- new net MOSI: JP3.3, U1.MOSI, U2.MOSI
- new net SCK: JP3.4, U1.SCK, U2.SCK
- net 3.3V: now also C2.1, C3.1, JP1.4, LED.A, MEM.A, R4.2, R5.2, U2.!HOLD, U2.!WP, U2.VCC; no longer ADDR.1, J1.2/VCC
- net GND: now also C2.2, J1.3, JP1.3, U2.GND; no longer ADDR.3, J1.12/GND, J1.14/GND, R4.1, U1.VPP
- net INT: now also JP2.2; no longer J1.28/IO2
- net N$1: now also MEM.C, U1.LED_IND; no longer C2.2, R4.2
- net N$2: now also LED.C, U1.LED_DRV; no longer C3.1, U1.DVDD-PC
- net N$3: now also J1.1, R5.1; no longer C2.1, U1.AVDD-PC
- net SCL: now also JP1.1, R1.1, U1.SCL/RX; no longer J1.1/SCL, R2.1, U1.SCL
- net SDA: now also JP1.2, R2.1, U1.SDA/TX; no longer J1.3/SDA, R1.1, U1.SDA
Other:
- moved on the sheet: C1, C2, C3, R1, R2, R3, R4
